File: cell2.kicad_sch (KiCad schematic)
At the start: 6 parts, among them Q3 SIS407DN-T1-GE3

Commit message: Replace broken 8-pin DMG2305UX symbol with correct 3-pin SamacSys version
- Updated lib_symbols with official DMG2305UX-7 symbol (G/S/D pins 1/2/3)
- Added SOT96P240X115-3N footprint file
- Applied to both cell.kicad_sch and cell2.kicad_sch

Note: Wire connections may need adjustment in KiCad GUI since pin geometry changed
Connections:
- net C+: no longer Q3.1 (S_1), Q3.2 (S_2), Q3.3 (S_3)
- net at R28.2: no longer Q3.4 (G)
- now unconnected: R29.2

Commit message: Adjust balancing resistor and balancing mosfet
Parts:
- removed Q3: SIS407DN-T1-GE3, Samacsys:SIS862DNT1GE3, symbol Samacsys:SIS407DN-T1-GE3
- removed R29: PWR263S-20-2R50J, Samacsys:PWR263S2010R0F, symbol Samacsys_kicad_sym:PWR263S-20-2R50J
- added Q3: DMG2305UX-7, Package_TO_SOT_SMD:SOT-23, symbol Samacsys:DMG2305UX-7
- added R29: 3.9, Resistor_SMD:R_2512_6332Metric, symbol Device:R
Connections:
- net C+: now also Q3.2 (S)
- net C-: now also R29.1
- net at R28.2: now also Q3.1 (G)
- new net: Q3.3 (D), R29.2
- no-connect marks 2 -> 0
